File: KiCad/Homework_SmartWatch_2/Homework_SmartWatch_2.kicad_sch (KiCad schematic)
At the start: 0 parts

Commit message: Add: L476RG: ST Morpho Connector
Parts:
- added U1: (no value), Nucleo:L476RG, symbol Nucleo:L476RG
Changed lines of the file:
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@@
 	(generator_version "10.0")
 	(paper "A4")
+	(symbol
+		(lib_id "Nucleo:L476RG")
+		(at 54.61 57.15 0)
+		(unit 1)
+		(body_style 1)
+		(exclude_from_sim no)
+		(in_bom yes)
+		(on_board yes)
+		(in_pos_files yes)
+		(dnp no)
+		(fields_autoplaced yes)
+		(property "Reference" "U1"
+			(at 54.61 33.02 0)
+			(show_name no)
+			(do_not_autoplace no)
+			(effects
+				(font
+					(size 1.27 1.27)
+				)
+			)
+		)
+		(property "Value" ""
+			(at 36.83 33.02 0)
+			(show_name no)
+			(do_not_autoplace no)
+			(effects
+				(font
+					(size 1.27 1.27)
+				)
+			)
+		)
+		(property "Footprint" "Nucleo:L476RG"
+			(at 36.83 33.02 0)
+			(hide yes)
+			(show_name no)
+			(do_not_autoplace no)
+			(effects
+				(font
+					(size 1.27 1.27)
+				)
+			)
+		)
+		(property "Datasheet" "./ref/um1724-stm32-nucleo64-boards-mb1136-stmicroelectronics.pdf"
+			(at 36.83 33.02 0)
+			(hide yes)
+			(show_name no)
+			(do_not_autoplace no)
+			(effects
+				(font
+					(size 1.27 1.27)
+				)
+			)
+		)
+		(property "Description" ""
+			(at 36.83 33.02 0)
+			(hide yes)
+			(show_name no)
+			(do_not_autoplace no)
+			(effects
+				(font
+					(size 1.27 1.27)
+				)
+			)
+		)
+		(pin "22"
+		)
+		(pin "28"
+		)
+		(pin "1"
+		)
+		(pin "0"
+		)
+		(pin "14"
+		)
+		(pin "2"
+		)
+		(pin "3"
+		)
+		(pin "23"
+		)
+		(pin "8"
+		)
+		(pin "19"
+		)
+		(pin "29"
+		)
+		(pin "12"
+		)
+		(pin "20"
+		)
+		(pin "15"
+		)
+		(pin "31"
+		)
+		(pin "9"
+		)
+		(pin "24"
+		)
+		(pin "25"
+		)
+		(pin "26"
+		)
+		(pin "30"
+		)
+		(pin "21"
+		)
+		(pin "10"
+		)
+		(pin "11"
+		)
+		(pin "27"
+		)
+		(pin "7"
+		)
+		(pin "16"
+		)
+		(pin "4"
+		)
+		(pin "18"
+		)
+		(pin "13"
+		)
+		(pin "17"
+		)
+		(pin "5"
+		)
+		(pin "6"
+		)
+		(instances
+			(project "Homework_SmartWatch_2"
+				(path "/28fd2d6b-5e74-43f0-9c9d-a7632017a632"
+					(reference "U1")
+					(unit 1)
+				)
+			)
+		)
+	)
 	(sheet_instances
 		(path "/"
